File: LogicBoard/LogicBoard.kicad_sch (KiCad schematic)
At the start: 57 parts, among them J1 Raspberry_Pi_4, J2 Screw_Terminal_01x04, J3 Screw_Terminal_01x04, J4 Screw_Terminal_01x08, J5 Screw_Terminal_01x04, J6 Screw_Terminal_01x06, J7 PINHD_1x4_Male, J8 Screw_Terminal_01x02, Q1 IRF520N, Q2 IRF520N, Q3 IRF520N, U1 STM32H743VITx, U2 MCP2557FD-xSN, U3 MCP2518FD-xQBB, U4 MCP2557FD-xSN, Y1-HSE1 830033075, Y2 ABS04W-32.768KHZ-LSE, Y3 ECS-400-9-36B-CKY-TR

Commit message: Prepared BOM, component placement file and minor changes to PCB
Parts:
- removed C14: 10uF, symbol PCM_Elektuur:C
- C15: value 10u -> 10uF
- C16, C17: value 1u -> 1uF
- C20, C21: value 25pF -> 24pF
- R13: renamed from 10k2; value R -> 10k
- Y1-HSE1: value 830033075 -> 7I25000F18UCG
- Y3: value ECS-400-9-36B-CKY-TR -> Q24FA20H00209
Changed lines of the file:
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@@
 	)
 	(junction
-		(at 257.81 39.37)
-		(diameter 0)
-		(color 0 0 0 0)
-	)
-	(junction
 		(at 59.69 238.76)
 		(diameter 0)
@@
 	(wire
 		(pts
-			(xy 254 39.37) (xy 257.81 39.37)
-		)
-		(stroke
-			(width 0)
-			(type default)
-		)
-	)
-	(wire
-		(pts
 			(xy 113.03 134.62) (xy 113.03 138.43)
 		)
@@
 	(wire
 		(pts
-			(xy 257.81 39.37) (xy 264.16 39.37)
+			(xy 254 39.37) (xy 264.16 39.37)
 		)
 		(stroke
@@
 		)
 	)
-	(wire
-		(pts
-			(xy 257.81 29.21) (xy 264.16 29.21)
-		)
-		(stroke
-			(width 0)
-			(type default)
-		)
-	)
 	(polyline
 		(pts
@@
 			)
 		)
-		(property "Value" "830033075"
+		(property "Value" "7I25000F18UCG"
 			(at 222.758 50.038 0)
 			(effects
@@
 		(on_board yes)
 		(dnp no)
-		(property "Reference" "10k2"
+		(property "Reference" "R13"
 			(at 287.274 58.674 90)
 			(effects
@@
 			)
 		)
-		(property "Value" "R"
+		(property "Value" "10k"
 			(at 287.02 55.88 90)
 			(do_not_autoplace yes)
@@
 			(project "LogicBoard"
 				(path "/48fa907e-ad89-429b-bed4-a3e0e90622bf"
-					(reference "10k2")
+					(reference "R13")
 					(unit 1)
 				)
@@
 			)
 		)
-		(property "Value" "ECS-400-9-36B-CKY-TR"
+		(property "Value" "Q24FA20H00209"
 			(at 22.352 160.528 0)
 			(effects
@@
 			)
 		)
-		(property "Value" "25pF"
+		(property "Value" "24pF"
 			(at 252.984 59.944 0)
 			(effects
@@
 	)
 	(symbol
-		(lib_id "PCM_Elektuur:C")
-		(at 257.81 34.29 0)
-		(unit 1)
-		(exclude_from_sim no)
-		(in_bom yes)
-		(on_board yes)
-		(dnp no)
-		(property "Reference" "C14"
-			(at 256.286 41.402 0)
-			(effects
-				(font
-					(size 1.27 1.27)
-				)
-				(justify left)
-			)
-		)
-		(property "Value" "10uF"
-			(at 256.286 43.942 0)
-			(effects
-				(font
-					(size 1.27 1.27)
-				)
-				(justify left)
-			)
-		)
-		(property "Footprint" ""
-			(at 257.81 34.29 0)
-			(effects
-				(font
-					(size 1.27 1.27)
-				)
-				(hide yes)
-			)
-		)
-		(property "Datasheet" ""
-			(at 257.81 34.29 0)
-			(effects
-				(font
-					(size 1.27 1.27)
-				)
-				(hide yes)
-			)
-		)
-		(property "Description" "capacitor, non-polarized/bipolar"
-			(at 257.81 34.29 0)
-			(effects
-				(font
-					(size 1.27 1.27)
-				)
-				(hide yes)
-			)
-		)
-		(property "Indicator" "+"
-			(at 256.54 31.115 0)
-			(do_not_autoplace yes)
-			(effects
-				(font
-					(size 1.27 1.27)
-				)
-				(hide yes)
-			)
-		)
-		(property "Rating" "V"
-			(at 257.175 37.465 0)
-			(effects
-				(font
-					(size 1.27 1.27)
-				)
-				(justify right)
-				(hide yes)
-			)
-		)
-		(pin "2"
-		)
-		(pin "1"
-		)
-		(instances
-			(project "LogicBoard"
-				(path "/48fa907e-ad89-429b-bed4-a3e0e90622bf"
-					(reference "C14")
-					(unit 1)
-				)
-			)
-		)
-	)
-	(symbol
 		(lib_id "power:GND")
 		(at 163.83 125.73 0)
@@
 			)
 		)
-		(property "Value" "25pF"
+		(property "Value" "24pF"
 			(at 202.184 75.184 0)
 			(effects
@@
 			)
 		)
-		(property "Value" "1u"
+		(property "Value" "1uF"
 			(at 365.76 33.02 0)
 			(effects
@@
 			)
 		)
-		(property "Value" "10u"
+		(property "Value" "10uF"
 			(at 359.156 32.258 0)
 			(effects
@@
 			)
 		)
-		(property "Value" "1u"
+		(property "Value" "1uF"
 			(at 382.27 33.02 0)
 			(effects

Commit message: Fix on LightColumn, added reverse-polarity protection, improved connectors, additional filtering lanes
Parts:
- removed J6: Screw_Terminal_01x06, symbol Connector:Screw_Terminal_01x06
- removed J7: PINHD_1x4_Male, Connector_PinHeader_2.54mm:PinHeader_1x04_P2.54mm_Vertical, symbol PCM_SL_Pin_Headers:PINHD_1x4_Male
- removed J8: Screw_Terminal_01x02, symbol Connector:Screw_Terminal_01x02
- removed Q2: IRF520N, PCM_Package_TO_SOT_THT_AKL:TO-220-3_Vertical_GDS, symbol PCM_Transistor_MOSFET_AKL:IRF520N
- added C14: 1uF, symbol PCM_Elektuur:C
- added C25, C26: 22uF, symbol PCM_Elektuur:C
- added D2, D3, D4: MMSZ5245BT1G, PCM_Diode_SMD_AKL:D_SOD-123F, symbol PCM_Diode_AKL:S07JFL
- added FB2: 120R at 100MHz, symbol PCM_Device_AKL:Ferrite_Bead
- added J10: XT30-3V3, symbol Connector:Conn_01x02_Socket
- added J6: Screw_Terminal_01x04, symbol Connector:Screw_Terminal_01x04
- added J7: XT30-5V, symbol Connector:Conn_01x02_Socket
- added J8: XT60-24V, symbol Connector:Conn_01x02_Socket
- added J9: PINHD_1x5_Male, Connector_PinHeader_2.54mm:PinHeader_1x05_P2.54mm_Vertical, symbol PCM_SL_Pin_Headers:PINHD_1x5_Male
- added LED1, LED2, LED3, LED4, LED5, LED6: LED_1206, PCM_LED_SMD_AKL:LED_1206_3216Metric, symbol PCM_LED_AKL:LED_1206
- added Q2, Q4, Q6: BCP56-16, PCM_Package_TO_SOT_SMD_AKL:SOT-223, symbol PCM_Transistor_BJT_AKL:BC547
- added Q5: FDT458P, PCM_Package_TO_SOT_SMD_AKL:SOT-223, symbol PCM_Transistor_MOSFET_AKL:IRF520N
- added R14, R22, R23, R25, R26, R27, R29: 10k, symbol PCM_Elektuur:R
- added R15, R18, R19, R20: 100, symbol PCM_Elektuur:R
- added R16: 200, symbol PCM_Elektuur:R
- added R17: 1k2, symbol PCM_Elektuur:R
- added R21, R24, R28: 2k2, symbol PCM_Elektuur:R
- added SW1: SW_Wuerth_450301014042, Button_Switch_THT:SW_Slide-03_Wuerth-WS-SLTV_10x2.5x6.4_P2.54mm, symbol Switch:SW_Wuerth_450301014042
- added SW2, SW3, SW4: CS22BNW03, CS22BNW03, symbol CS22BNW03:CS22BNW03
- added TP1, TP2, TP3, TP4, TP5, TP6: TestPoint, symbol Connector:TestPoint
- C18: value 100nF -> 10uF
- Q1, Q3: value IRF520N -> FDT458P; footprint PCM_Package_TO_SOT_THT_AKL:TO-220-3_Vertical_GDS -> PCM_Package_TO_SOT_SMD_AKL:SOT-223
- renumbered Z1 to D1
Connections:
- net +24V: now also D2.1 (K), D3.1 (K), D4.1 (K), LED3.2 (A), Q5.3 (S), R22.1 (+), R23.1 (+), R25.1 (+), SW2.2 (COM_1), TP1.1
- net +3V3: now also J9.1, LED1.2 (A), SW1.3 (A), SW4.2 (COM_1), TP3.1
- net +5V: now also LED2.2 (A), SW3.2 (COM_1), TP2.1
- net DEBUG_SWCLK: now also J9.3
- net DEBUG_SWDIO: now also J9.2
- net GND: now also C14.1 (+), C25.1 (+), C26.1 (+), J10.2 (Pin_2), J6.4 (Pin_4), J7.2 (Pin_2), J8.2 (Pin_2), J9.5, Q2.1 (C), Q4.1 (C), Q6.1 (C), R15.2 (-), R16.2 (-), R17.2 (-), R18.2 (-), R19.2 (-), R20.2 (-), R26.1 (+), R27.1 (+), R29.1 (+), SW2.4 (NC_2), SW2.5 (COM_2), SW2.6 (NO_2), SW3.4 (NC_2), SW3.5 (COM_2), SW3.6 (NO_2), SW4.4 (NC_2), SW4.5 (COM_2), SW4.6 (NO_2), TP4.1
- net GreenLight_Modulated: now also Q3.2 (D), J6.1 (Pin_1); no longer Q1.2 (D)
- net RedLight_Modulated: now also Q1.2 (D), J6.3 (Pin_3); no longer Q3.2 (D)
- net TIM13: now also R24.1 (+); no longer Q1.1 (G), Q3.1 (G)
- net TIM14: now also R28.1 (+)
- net TIM15: now also R21.1 (+)
- net YellowLight_Modulated: now also J6.2 (Pin_2), Q5.2 (D)
- net at U1.14 (NRST): now also R14.1 (+); no longer C18.2 (-)
- net CANActivity: now reaches U1.36 (PB2)
- net CANActivity: now also LED6.2 (A)
- net StatusLED: now reaches U1.37 (PE7)
- net StatusLED: now also LED5.2 (A)
- net HeartBeat: now reaches U1.38 (PE8)
- net HeartBeat: now also LED4.2 (A)
- net CanL: now reaches R4.2 (-), R8.1 (+), U2.6 (CANL), U4.6 (CANL)
- net CanL: now also TP5.1
- net CanH: now reaches R5.1 (+), R9.2 (-), U2.7 (CANH), U4.7 (CANH)
- net CanH: now also TP6.1
- new net: LED6.1 (K), R20.1 (+)
- new net: C26.2 (-), J7.1 (Pin_1), SW3.1 (NC_1)
- new net: LED5.1 (K), R19.1 (+)
- new net: C14.2 (-), R14.2 (-), SW1.1 (B)
- new net: Q2.2 (B), R21.2 (-)
- new net: D4.2 (A), Q5.1 (G), Q6.3 (E), R23.2 (-)
- new net: C18.2 (-), C25.2 (-), FB2.1, SW4.1 (NC_1)
- new net: D3.2 (A), Q1.1 (G), Q2.3 (E), R22.2 (-)
- new net: Q6.2 (B), R28.2 (-), R29.2 (-)
- new net: LED4.1 (K), R18.1 (+)
- new net: J8.1 (Pin_1), SW2.1 (NC_1)
- new net: LED2.1 (K), R16.1 (+)
- new net: LED3.1 (K), R17.1 (+)
- new net: FB2.2, J10.1 (Pin_1)
- new net: Q4.2 (B), R24.2 (-), R26.2 (-)
- new net: LED1.1 (K), R15.1 (+)
- new net: D2.2 (A), Q3.1 (G), Q4.3 (E), R25.2 (-)
- new net DEBUG_RST: J9.4, SW1.2 (C)
Other:
- note added: "24V BUS ACTIV"
- note added: "3V3 BUS ACTIV"
- note added: "5V BUS ACTIV"
- note added: "ADD. FILTERING"
- note added: "CAN ACTIV"
- note added: "EXT. 24V"
- note added: "EXT. 3V3"
- note added: "EXT. 5V"
- note added: "FE-PWM Z AXIS WHEELS"
- note added: "MCU ACTIV"
- note added: "STATUS"
- note added: "TEST POINT DEBUG"
- note added: "VISUAL DEBUG"
- note removed: "FE - PWM Z AXIS WHEELS"
- moved on the sheet: J5

Commit message: Fixes to tags, nets and silkscreen
Parts:
- C1, C2: value 14pF -> 12pF
- C19, C22: value 6pF -> 8pF
- C20, C21: value 24pF -> 27pF
- R11: value 80k -> 100k
- R12: value 10k -> 12k
- Y1-HSE1: value 7I25000F18UCG -> 830033075
- Y3: value Q24FA20H00209 -> ECS400936BCKYTR
- renumbered FB11 to FB1
Changed lines of the file:
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@@
 			)
 		)
-		(property "Value" "6pF"
+		(property "Value" "8pF"
 			(at 368.3 180.34 90)
 			(effects
@@
 			)
 		)
-		(property "Value" "7I25000F18UCG"
+		(property "Value" "830033075"
 			(at 222.758 50.038 0)
 			(effects
@@
 		(on_board yes)
 		(dnp no)
-		(property "Reference" "FB11"
+		(property "Reference" "FB1"
 			(at 375.92 31.75 0)
 			(effects
@@
 			(project "LogicBoard"
 				(path "/48fa907e-ad89-429b-bed4-a3e0e90622bf"
-					(reference "FB11")
+					(reference "FB1")
 					(unit 1)
 				)
@@
 			)
 		)
-		(property "Value" "10k"
+		(property "Value" "12k"
 			(at 19.05 246.38 90)
 			(do_not_autoplace yes)
@@
 			)
 		)
-		(property "Value" "Q24FA20H00209"
+		(property "Value" "ECS400936BCKYTR"
 			(at 22.352 160.528 0)
 			(effects
@@
 			)
 		)
-		(property "Value" "24pF"
+		(property "Value" "27pF"
 			(at 251.206 63.754 0)
 			(effects
@@
 			)
 		)
-		(property "Value" "14pF"
+		(property "Value" "12pF"
 			(at 39.37 185.42 90)
 			(effects
@@
 			)
 		)
-		(property "Value" "6pF"
+		(property "Value" "8pF"
 			(at 391.922 156.464 0)
 			(effects
@@
 			)
 		)
-		(property "Value" "24pF"
+		(property "Value" "27pF"
 			(at 202.184 75.184 0)
 			(effects
@@
 			)
 		)
-		(property "Value" "14pF"
+		(property "Value" "12pF"
 			(at 21.59 151.13 90)
 			(effects
@@
 			)
 		)
-		(property "Value" "80k"
+		(property "Value" "100k"
 			(at 19.05 232.41 90)
 			(do_not_autoplace yes)
